File: LinuxRulerHardware.kicad_sch (KiCad schematic)
At the start: 0 parts

Commit message: file sync
Other:
- removed sheet [1] - SoC Power And Configurations
- removed sheet [2] - DDR SDRAM
- removed sheet [3] - NAND Flash
- removed sheet [4] - Screen Controller
- removed sheet [5] - Power Supply
- added sheet [1] - Battery Charge (bc.kicad_sch)
- added sheet [1] - SoC-PWR (RK_PWR.kicad_sch)
Changed lines of the file:
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@@
-(kicad_sch (version 20221206) (generator eeschema)
+(kicad_sch (version 20230121) (generator eeschema)
   (paper "A4")
-  (sheet (at 13.97 165.735) (size 44.45 28.575) (fields_autoplaced)
+  (sheet (at 19.685 161.29) (size 49.53 29.21) (fields_autoplaced)
     (stroke (width 0.1524) (type solid))
     (fill (color 0 0 0 0.0000))
-    (property "Sheetname" "[1] - SoC Power And Configurations" (at 13.97 165.0234 0)
+    (property "Sheetname" "[1] - Battery Charge" (at 19.685 160.5784 0)
       (effects (font (size 1.27 1.27)) (justify left bottom))
     )
-    (property "Sheetfile" "soc_pwr.kicad_sch" (at 13.97 194.8946 0)
-      (effects (font (size 1.27 1.27)) (justify left top))
-    )
-    (instances
-      (project "LinuxRulerHardware"
-        (path "/139c7518-bdce-4d72-a2f4-8829476221aa" (page "2"))
-      )
-    )
-  )
-  (sheet (at 61.595 165.735) (size 45.72 28.575) (fields_autoplaced)
-    (stroke (width 0.1524) (type solid))
-    (fill (color 0 0 0 0.0000))
-    (property "Sheetname" "[2] - DDR SDRAM" (at 61.595 165.0234 0)
-      (effects (font (size 1.27 1.27)) (justify left bottom))
-    )
-    (property "Sheetfile" "ddr.kicad_sch" (at 61.595 194.8946 0)
+    (property "Sheetfile" "bc.kicad_sch" (at 19.685 191.0846 0)
       (effects (font (size 1.27 1.27)) (justify left top))
     )
@@
     )
   )
-  (sheet (at 61.595 128.905) (size 45.72 30.48) (fields_autoplaced)
+  (sheet (at 15.875 15.875) (size 46.355 28.575) (fields_autoplaced)
     (stroke (width 0.1524) (type solid))
     (fill (color 0 0 0 0.0000))
-    (property "Sheetname" "[5] - Power Supply" (at 61.595 128.1934 0)
+    (property "Sheetname" "[1] - SoC-PWR" (at 15.875 15.1634 0)
       (effects (font (size 1.27 1.27)) (justify left bottom))
     )
-    (property "Sheetfile" "power.kicad_sch" (at 61.595 159.9696 0)
+    (property "Sheetfile" "RK_PWR.kicad_sch" (at 15.875 45.0346 0)
       (effects (font (size 1.27 1.27)) (justify left top))
     )
     (instances
       (project "LinuxRulerHardware"
-        (path "/139c7518-bdce-4d72-a2f4-8829476221aa" (page "6"))
+        (path "/139c7518-bdce-4d72-a2f4-8829476221aa" (page "2"))
       )
     )
-  )
-  (sheet (at 109.855 165.735) (size 45.085 28.575) (fields_autoplaced)
-    (stroke (width 0.1524) (type solid))
-    (fill (color 0 0 0 0.0000))
-    (property "Sheetname" "[3] - NAND Flash" (at 109.855 165.0234 0)
-      (effects (font (size 1.27 1.27)) (justify left bottom))
-    )
-    (property "Sheetfile" "nand-flash.kicad_sch" (at 109.855 194.8946 0)
-      (effects (font (size 1.27 1.27)) (justify left top))
-    )
-    (instances
-      (project "LinuxRulerHardware"
-        (path "/139c7518-bdce-4d72-a2f4-8829476221aa" (page "4"))
-      )
-    )
-  )
-  (sheet (at 13.97 128.905) (size 44.45 30.48) (fields_autoplaced)
-    (stroke (width 0.1524) (type solid))
-    (fill (color 0 0 0 0.0000))
-    (property "Sheetname" "[4] - Screen Controller" (at 13.97 128.1934 0)
-      (effects (font (size 1.27 1.27)) (justify left bottom))
-    )
-    (property "Sheetfile" "screen.kicad_sch" (at 13.97 159.9696 0)
-      (effects (font (size 1.27 1.27)) (justify left top))
-    )
-    (instances
-      (project "LinuxRulerHardware"
-        (path "/139c7518-bdce-4d72-a2f4-8829476221aa" (page "5"))
-      )
-    )

Commit message: DDR sch
Other:
- added sheet [2] - DDR (ddr.kicad_sch)
Changed lines of the file:
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@@
+    )
+  )
+  (sheet (at 71.755 16.51) (size 43.815 28.575) (fields_autoplaced)
+    (stroke (width 0.1524) (type solid))
+    (fill (color 0 0 0 0.0000))
+    (property "Sheetname" "[2] - DDR" (at 71.755 15.7984 0)
+      (effects (font (size 1.27 1.27)) (justify left bottom))
+    )
+    (property "Sheetfile" "ddr.kicad_sch" (at 71.755 45.6696 0)
+      (effects (font (size 1.27 1.27)) (justify left top))
+    )
+    (instances
+      (project "LinuxRulerHardware"
+        (path "/139c7518-bdce-4d72-a2f4-8829476221aa" (page "4"))
+      )
     )
   )

Commit message: file sync
Other:
- added sheet [2] - Power Management (pm.kicad_sch)
- added sheet [3] - NAND Flash (flash.kicad_sch)
Changed lines of the file:
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@@
+    )
+  )
+  (sheet (at 72.39 161.29) (size 99.695 29.21) (fields_autoplaced)
+    (stroke (width 0.1524) (type solid))
+    (fill (color 0 0 0 0.0000))
+    (property "Sheetname" "[2] - Power Management" (at 72.39 160.5784 0)
+      (effects (font (size 1.27 1.27)) (justify left bottom))
+    )
+    (property "Sheetfile" "pm.kicad_sch" (at 72.39 191.0846 0)
+      (effects (font (size 1.27 1.27)) (justify left top))
+    )
+    (instances
+      (project "LinuxRulerHardware"
+        (path "/139c7518-bdce-4d72-a2f4-8829476221aa" (page "6"))
+      )
     )
   )
@@
     )
   )
-  (sheet (at 71.755 16.51) (size 43.815 28.575) (fields_autoplaced)
+  (sheet (at 130.81 15.875) (size 59.055 28.575) (fields_autoplaced)
     (stroke (width 0.1524) (type solid))
     (fill (color 0 0 0 0.0000))
-    (property "Sheetname" "[2] - DDR" (at 71.755 15.7984 0)
+    (property "Sheetname" "[3] - NAND Flash" (at 130.81 15.1634 0)
       (effects (font (size 1.27 1.27)) (justify left bottom))
     )
-    (property "Sheetfile" "ddr.kicad_sch" (at 71.755 45.6696 0)
+    (property "Sheetfile" "flash.kicad_sch" (at 130.81 45.0346 0)
       (effects (font (size 1.27 1.27)) (justify left top))
     )
+    (instances
+      (project "LinuxRulerHardware"
+        (path "/139c7518-bdce-4d72-a2f4-8829476221aa" (page "5"))
+      )
+    )
+  )
+  (sheet (at 71.755 15.875) (size 49.53 28.575) (fields_autoplaced)
+    (stroke (width 0.1524) (type solid))
+    (fill (color 0 0 0 0.0000))
+    (property "Sheetname" "[2] - DDR" (at 71.755 15.1634 0)
+      (effects (font (size 1.27 1.27)) (justify left bottom))
+    )
+    (property "Sheetfile" "ddr.kicad_sch" (at 71.755 45.0346 0)
+      (effects (font (size 1.27 1.27)) (justify left top))
+    )
