File: bc.kicad_sch (KiCad schematic)
At the start: 22 parts, among them J1 Conn_01x02_Pin, P1 USB_C_Plug_USB2.0, U2 BQ25606

Commit message: file sync
Connections:
- net GND: now also J1.2 (Pin_2)
- net +BATT: now reaches U2.13 (BAT)
- net +BATT: now also J1.1 (Pin_1), U2.14 (BAT); no longer J1.2 (Pin_2)
Changed lines of the file:
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@@
   (junction (at 98.425 43.18) (diameter 0) (color 0 0 0 0)
   )
+  (junction (at 67.31 50.8) (diameter 0) (color 0 0 0 0)
+  )
   (junction (at 102.235 43.18) (diameter 0) (color 0 0 0 0)
   )
@@
   )
   (junction (at 88.9 40.64) (diameter 0) (color 0 0 0 0)
+  )
+  (junction (at 68.58 53.34) (diameter 0) (color 0 0 0 0)
   )
   (junction (at 88.9 35.56) (diameter 0) (color 0 0 0 0)
@@
     (stroke (width 0) (type default))
   )
+  (wire (pts (xy 67.31 50.8) (xy 68.58 50.8))
+    (stroke (width 0) (type default))
+  )
   (wire (pts (xy 51.435 44.45) (xy 40.005 44.45))
     (stroke (width 0) (type default))
@@
     (stroke (width 0) (type default))
   )
+  (wire (pts (xy 66.04 53.34) (xy 66.04 53.975))
+    (stroke (width 0) (type default))
+  )
   (wire (pts (xy 88.9 48.26) (xy 90.805 48.26))
     (stroke (width 0) (type default))
@@
     (stroke (width 0) (type default))
   )
+  (wire (pts (xy 68.58 53.34) (xy 67.31 53.34))
+    (stroke (width 0) (type default))
+  )
+  (wire (pts (xy 67.31 50.8) (xy 67.31 53.34))
+    (stroke (width 0) (type default))
+  )
   (wire (pts (xy 67.945 48.26) (xy 68.58 48.26))
     (stroke (width 0) (type default))
   )
-  (wire (pts (xy 64.77 50.8) (xy 68.58 50.8))
+  (wire (pts (xy 64.77 50.8) (xy 67.31 50.8))
     (stroke (width 0) (type default))
   )
@@
     (stroke (width 0) (type default))
   )
+  (wire (pts (xy 64.77 53.34) (xy 66.04 53.34))
+    (stroke (width 0) (type default))
+  )
   (wire (pts (xy 51.435 43.18) (xy 51.435 44.45))
-    (stroke (width 0) (type default))
-  )
-  (wire (pts (xy 64.77 53.34) (xy 68.58 53.34))
     (stroke (width 0) (type default))
   )
@@
         (path "/139c7518-bdce-4d72-a2f4-8829476221aa/1bc055cb-4072-4f8f-a1c9-26818f7ca321"
           (reference "R3") (unit 1)
+        )
+      )
+    )
+  )
+  (symbol (lib_id "power:GND") (at 66.04 53.975 0) (unit 1)
+    (in_bom yes) (on_board yes) (dnp no) (fields_autoplaced)
+    (property "Reference" "#PWR045" (at 66.04 60.325 0)
+      (effects (font (size 1.27 1.27)) hide)
+    )
+    (property "Value" "GND" (at 66.04 58.42 0)
+      (effects (font (size 1.27 1.27)) hide)
+    )
+    (property "Footprint" "" (at 66.04 53.975 0)
+      (effects (font (size 1.27 1.27)) hide)
+    )
+    (property "Datasheet" "" (at 66.04 53.975 0)
+      (effects (font (size 1.27 1.27)) hide)
+    )
+    (pin "1")
+    (instances
+      (project "LinuxRulerHardware"
+        (path "/139c7518-bdce-4d72-a2f4-8829476221aa/1bc055cb-4072-4f8f-a1c9-26818f7ca321"
+          (reference "#PWR045") (unit 1)
         )
       )
@@
         )
       )
+    )
+  )
+  (symbol (lib_id "power:+BATT") (at 68.58 53.34 180) (unit 1)
+    (in_bom yes) (on_board yes) (dnp no)
+    (property "Reference" "#PWR044" (at 68.58 49.53 0)
+      (effects (font (size 1.27 1.27)) hide)
+    )
+    (property "Value" "+BATT" (at 70.485 55.245 0)
+      (effects (font (size 0.64 0.64)))
+    )
+    (property "Footprint" "" (at 68.58 53.34 0)
+      (effects (font (size 1.27 1.27)) hide)
+    )
+    (property "Datasheet" "" (at 68.58 53.34 0)
+      (effects (font (size 1.27 1.27)) hide)
+    )
+    (pin "1")
+    (instances
+      (project "LinuxRulerHardware"
+        (path "/139c7518-bdce-4d72-a2f4-8829476221aa/1bc055cb-4072-4f8f-a1c9-26818f7ca321"
+          (reference "#PWR044") (unit 1)
+        )
+      )
