File: ddr.kicad_sch (KiCad schematic)
At the start: 32 parts, among them U2 K4B4G1646Q, U3 K4B4G1646Q

Commit message: DDR sch
Parts:
- removed U1: ~, Library:BGA-441_21x21_14.0x14.0mm, symbol Symbols:RK3326
- added U1: ~, symbol Symbols:RK3128
Connections:
- net +1V5: now also U1.G11 (DDR_VDD), U1.G8 (DDR_VDD), U1.G9 (DDR_VDD), U1.H7 (DDR_VDD), U1.J7 (DDR_VDD), U1.L7 (DDR_VDD), U1.M7 (DDR_VDD)
- net A0: now also U1.D1 (DDR_A0)
- net A1: now also U1.A4 (DDR_A1)
- net A10: now also U1.C4 (DDR_A10)
- net A11: now also U1.C5 (DDR_A11)
- net A12: now also U1.B4 (DDR_A12)
- net A13: now also U1.G1 (DDR_A13)
- net A14: now also U1.B5 (DDR_A14)
- net A2: now also U1.E2 (DDR_A2)
- net A3: now also U1.D2 (DDR_A3)
- net A4: now also U1.A2 (DDR_A4)
- net A5: now also U1.E5 (DDR_A5)
- net A6: now also U1.F7 (DDR_A6)
- net A7: now also U1.E4 (DDR_A7)
- net A8: now also U1.D8 (DDR_A8)
- net A9: now also U1.E1 (DDR_A9)
- net BA0: now also U1.D7 (DDR_BA0)
- net BA1: now also U1.E8 (DDR_BA1)
- net BA2: now also U1.D3 (DDR_BA2)
- net CASN: now also U1.E7 (DDR_CASN)
- net CKE: now also U1.B3 (DDR_CKE)
- net D0: now also U2.F2 (DQ2), U1.A14 (DDR_DQ0); no longer U2.A7 (DQ12)
- net D1: now also U2.H8 (DQ5), U1.F8 (DDR_DQ1); no longer U2.C3 (DQ9)
- net D10: now also U3.H8 (DQ5), U1.F2 (DDR_DQ10); no longer U2.F7 (DQ1)
- net D11: now also U3.E3 (DQ0), U1.H6 (DDR_DQ11); no longer U2.E3 (DQ0)
- net D12: now also U3.H3 (DQ4), U1.H3 (DDR_DQ12); no longer U2.H7 (DQ7)
- net D13: now also U3.F7 (DQ1), U1.J2 (DDR_DQ13); no longer U2.H3 (DQ4)
- net D14: now also U3.G2 (DQ6), U1.K2 (DDR_DQ14); no longer U2.H8 (DQ5)
- net D15: now also U3.F2 (DQ2), U1.K1 (DDR_DQ15); no longer U2.F2 (DQ2)
- net D16: now also U2.D7 (DQ8), U1.A10 (DDR_DQ16); no longer U3.A2 (DQ13)
- net D17: now also U2.A7 (DQ12), U1.C11 (DDR_DQ17); no longer U3.C3 (DQ9)
- net D18: now also U2.B8 (DQ14), U1.B9 (DDR_DQ18); no longer U3.A3 (DQ15)
- net D19: now also U2.A2 (DQ13), U1.E11 (DDR_DQ19); no longer U3.A7 (DQ12)
- net D2: now also U2.H7 (DQ7), U1.F11 (DDR_DQ2); no longer U2.D7 (DQ8)
- net D20: now also U2.C3 (DQ9), U1.E10 (DDR_DQ20); no longer U3.B8 (DQ14)
- net D21: now also U2.C8 (DQ10), U1.B12 (DDR_DQ21); no longer U3.D7 (DQ8)
- net D22: now also U2.C2 (DQ11), U1.F10 (DDR_DQ22); no longer U3.C2 (DQ11)
- net D23: now also U2.A3 (DQ15), U1.A13 (DDR_DQ23); no longer U3.C8 (DQ10)
- net D24: now also U3.D7 (DQ8), U1.K4 (DDR_DQ24); no longer U3.H7 (DQ7)
- net D25: now also U3.C3 (DQ9), U1.L4 (DDR_DQ25); no longer U3.F8 (DQ3)
- net D26: now also U3.C8 (DQ10), U1.G4 (DDR_DQ26); no longer U3.H3 (DQ4)
- net D27: now also U3.A2 (DQ13), U1.K5 (DDR_DQ27); no longer U3.G2 (DQ6)
- net D28: now also U3.A7 (DQ12), U1.H5 (DDR_DQ28); no longer U3.H8 (DQ5)
- net D29: now also U3.A3 (DQ15), U1.K6 (DDR_DQ29); no longer U3.F7 (DQ1)
- net D3: now also U2.F8 (DQ3), U1.A7 (DDR_DQ3); no longer U2.C8 (DQ10)
- net D30: now also U3.B8 (DQ14), U1.L5 (DDR_DQ30); no longer U3.F2 (DQ2)
- net D31: now also U3.C2 (DQ11), U1.L6 (DDR_DQ31); no longer U3.E3 (DQ0)
- net D4: now also U2.F7 (DQ1), U1.B10 (DDR_DQ4); no longer U2.C2 (DQ11)
- net D5: now also U2.H3 (DQ4), U1.D10 (DDR_DQ5); no longer U2.A2 (DQ13)
- net D6: now also U2.E3 (DQ0), U1.B13 (DDR_DQ6); no longer U2.A3 (DQ15)
- net D7: now also U2.G2 (DQ6), U1.C8 (DDR_DQ7); no longer U2.B8 (DQ14)
- net D8: now also U3.H7 (DQ7), U1.G6 (DDR_DQ8); no longer U2.F8 (DQ3)
- net D9: now also U3.F8 (DQ3), U1.G5 (DDR_DQ9); no longer U2.G2 (DQ6)
- net DDR_CLKN: now also U1.C2 (DDR_CLKN)
- net DDR_CLKP: now also U1.B1 (DDR_CLKP)
- net DDR_CS0N: now also U1.A1 (DDR_CS0)
- net DDR_CS1N: now also U1.B6 (DDR_CS1)
- net DDR_RST: now also U1.F6 (DDR_RST)
- net DM0: now also U1.B7 (DDR_DM0)
- net DM1: now also U1.H4 (DDR_DM1)
- net DM2: now also U1.D11 (DDR_DM2)
- net DM3: now also U1.L3 (DDR_DM3)
- net DQS0N: now also U1.B8 (DDR_DQS0N)
- net DQS0P: now also U1.A8 (DDR_DQS0P)
- net DQS1N: now also U1.H2 (DDR_DQS1N)
- net DQS1P: now also U1.H1 (DDR_DQS1P)
- net DQS2N: now also U1.B11 (DDR_DQS2N)
- net DQS2P: now also U1.A11 (DDR_DQS2P)
- net DQS3N: now also U1.L2 (DDR_DQS3N)
- net DQS3P: now also U1.L1 (DDR_DQS3P)
- net ODT0: now also U1.B2 (DDR_ODT0)
- net ODT1: now also U1.G2 (DDR_ODT1)
- net RASN: now also U1.E3 (DDR_RASN)
- net WEN: now also U1.D5 (DDR_WEN)

Commit message: file sync
Other:
- moved on the sheet: U1C
